Commit message: Merge branch 'feature/designCost'

File: mlivr_description/urdf/ur5e/ur5e_macro.xacro (robot description, xacro)
@@ -1,5 +1,5 @@
 <?xml version="1.0" encoding="utf-8"?>
 <robot xmlns:xacro="http://ros.org/wiki/xacro">
-  <xacro:property name="joint_damping" value="0.5" />
+  <xacro:property name="joint_damping" value="0.1" />
   <xacro:macro name="ur5e" params="prefix parent *origin">
     <joint name="${prefix}_base_joint" type="fixed">
