Commit message: Change robot base and gripper color

File: mlivr_description/urdf/ur5e/mlivr.xacro (robot description, xacro)
@@ -17,6 +17,6 @@
         <box size="0.2 0.2 0.2"/>
       </geometry>
-      <material name="gray">
-        <color rgba="0.5 0.5 0.5 1.0"/>
+      <material name="">
+        <color rgba="0.9 0.9 0.9 1.0"/>
       </material>
     </visual>

File: mlivr_description/urdf/ur5e/mlivr_gripper.xacro (robot description, xacro)
@@ -26,6 +26,6 @@
           <cylinder radius="0.03" length="0.05"/>
         </geometry>
-        <material name="gray">
-          <color rgba="0.5 0.5 0.5 1.0"/>
+        <material name="">
+          <color rgba="0.9 0.9 0.9 1.0"/>
         </material>
       </visual>
