Commit message: Merge branch 'feature/changeRobotModel'

File: mlivr_description/urdf/mlivr.urdf (robot description, URDF)
Before this commit: robot MLIVR, 21 links, 20 joints
Links:
- removed link limb_1_link_0
- removed link limb_1_link_1
- removed link limb_1_link_2
- removed link limb_1_link_3
- removed link limb_1_link_4
- removed link limb_1_link_5
- removed link limb_1_link_6
- removed link limb_1_link_7
- removed link limb_1_link_ee
- removed link limb_1_link_gripper
- removed link limb_2_link_0
- removed link limb_2_link_1
- removed link limb_2_link_2
- removed link limb_2_link_3
- removed link limb_2_link_4
- removed link limb_2_link_5
- removed link limb_2_link_6
- removed link limb_2_link_7
- removed link limb_2_link_ee
- removed link limb_2_link_gripper
- added link limb_1_base_link, mass 4.0; collision mesh filename=../meshes/ur5e/collision/base.stl scale=1.0 1.0 1.0; visual mesh filename=../meshes/ur5e/visual/base.dae
- added link limb_1_ee_link; collision box size=0.01 0.01 0.01
- added link limb_1_forearm_link, mass 2.275; collision mesh filename=../meshes/ur5e/collision/forearm.stl scale=1.0 1.0 1.0; visual mesh filename=../meshes/ur5e/visual/forearm.dae
- added link limb_1_shoulder_link, mass 3.7; collision mesh filename=../meshes/ur5e/collision/shoulder.stl scale=1.0 1.0 1.0; visual mesh filename=../meshes/ur5e/visual/shoulder.dae
- added link limb_1_tool0
- added link limb_1_upper_arm_link, mass 8.393; collision mesh filename=../meshes/ur5e/collision/upperarm.stl scale=1.0 1.0 1.0; visual mesh filename=../meshes/ur5e/visual/upperarm.dae
- added link limb_1_wrist_1_link, mass 1.219; collision mesh filename=../meshes/ur5e/collision/wrist1.stl scale=1.0 1.0 1.0; visual mesh filename=../meshes/ur5e/visual/wrist1.dae
- added link limb_1_wrist_2_link, mass 1.219; collision mesh filename=../meshes/ur5e/collision/wrist2.stl scale=1.0 1.0 1.0; visual mesh filename=../meshes/ur5e/visual/wrist2.dae
- added link limb_1_wrist_3_link, mass 0.1879; collision mesh filename=../meshes/ur5e/collision/wrist3.stl scale=1.0 1.0 1.0; visual mesh filename=../meshes/ur5e/visual/wrist3.dae
- added link limb_2_base_link, mass 4.0; collision mesh filename=../meshes/ur5e/collision/base.stl scale=1.0 1.0 1.0; visual mesh filename=../meshes/ur5e/visual/base.dae
- added link limb_2_ee_link; collision box size=0.01 0.01 0.01
- added link limb_2_forearm_link, mass 2.275; collision mesh filename=../meshes/ur5e/collision/forearm.stl scale=1.0 1.0 1.0; visual mesh filename=../meshes/ur5e/visual/forearm.dae
- added link limb_2_shoulder_link, mass 3.7; collision mesh filename=../meshes/ur5e/collision/shoulder.stl scale=1.0 1.0 1.0; visual mesh filename=../meshes/ur5e/visual/shoulder.dae
- added link limb_2_tool0
- added link limb_2_upper_arm_link, mass 8.393; collision mesh filename=../meshes/ur5e/collision/upperarm.stl scale=1.0 1.0 1.0; visual mesh filename=../meshes/ur5e/visual/upperarm.dae
- added link limb_2_wrist_1_link, mass 1.219; collision mesh filename=../meshes/ur5e/collision/wrist1.stl scale=1.0 1.0 1.0; visual mesh filename=../meshes/ur5e/visual/wrist1.dae
- added link limb_2_wrist_2_link, mass 1.219; collision mesh filename=../meshes/ur5e/collision/wrist2.stl scale=1.0 1.0 1.0; visual mesh filename=../meshes/ur5e/visual/wrist2.dae
- added link limb_2_wrist_3_link, mass 0.1879; collision mesh filename=../meshes/ur5e/collision/wrist3.stl scale=1.0 1.0 1.0; visual mesh filename=../meshes/ur5e/visual/wrist3.dae
- link base_link: mass 50.0 -> 30.0; geometry collision box size=0.2 0.2 0.2; visual box size=0.2 0.2 0.2
Joints:
- removed joint base_link_limb_1_joint
- removed joint base_link_limb_2_joint
- removed joint limb_1_joint_1
- removed joint limb_1_joint_2
- removed joint limb_1_joint_3
- removed joint limb_1_joint_4
- removed joint limb_1_joint_5
- removed joint limb_1_joint_6
- removed joint limb_1_joint_7
- removed joint limb_1_joint_ee
- removed joint limb_1_joint_gripper
- removed joint limb_2_joint_1
- removed joint limb_2_joint_2
- removed joint limb_2_joint_3
- removed joint limb_2_joint_4
- removed joint limb_2_joint_5
- removed joint limb_2_joint_6
- removed joint limb_2_joint_7
- removed joint limb_2_joint_ee
- removed joint limb_2_joint_gripper
- added joint limb_1_base_joint: type fixed, parent base_link, child limb_1_base_link, origin xyz=0.0 0.1 0.0 rpy=0 1.5707963267948966 1.5707963267948966
- added joint limb_1_ee_fixed_joint: type fixed, parent limb_1_wrist_3_link, child limb_1_ee_link, origin xyz=0.0 0.1 0.0 rpy=0.0 0.0 1.57079632679
- added joint limb_1_elbow_joint: type revolute, parent limb_1_upper_arm_link, child limb_1_forearm_link, origin xyz=0.0 -0.131 0.425 rpy=0.0 0.0 0.0, axis 0 1 0, limit lower=-3.14159265359 upper=3.14159265359 effort=150.0 velocity=3.14
- added joint limb_1_shoulder_lift_joint: type revolute, parent limb_1_shoulder_link, child limb_1_upper_arm_link, origin xyz=0.0 0.138 0.0 rpy=0.0 1.57079632679 0.0, axis 0 1 0, limit lower=-6.28318530718 upper=6.28318530718 effort=150.0 velocity=3.14
- added joint limb_1_shoulder_pan_joint: type revolute, parent limb_1_base_link, child limb_1_shoulder_link, origin xyz=0.0 0.0 0.163 rpy=0.0 0.0 0.0, axis 0 0 1, limit lower=-6.28318530718 upper=6.28318530718 effort=150.0 velocity=3.14
- added joint limb_1_wrist_1_joint: type revolute, parent limb_1_forearm_link, child limb_1_wrist_1_link, origin xyz=0.0 0.0 0.392 rpy=0.0 1.57079632679 0.0, axis 0 1 0, limit lower=-6.28318530718 upper=6.28318530718 effort=28.0 velocity=6.28
- added joint limb_1_wrist_2_joint: type revolute, parent limb_1_wrist_1_link, child limb_1_wrist_2_link, origin xyz=0.0 0.127 0.0 rpy=0.0 0.0 0.0, axis 0 0 1, limit lower=-6.28318530718 upper=6.28318530718 effort=28.0 velocity=6.28
- added joint limb_1_wrist_3_joint: type revolute, parent limb_1_wrist_2_link, child limb_1_wrist_3_link, origin xyz=0.0 0.0 0.1 rpy=0.0 0.0 0.0, axis 0 1 0, limit lower=-6.28318530718 upper=6.28318530718 effort=28.0 velocity=6.28
- added joint limb_1_wrist_3_link-tool0_fixed_joint: type fixed, parent limb_1_wrist_3_link, child limb_1_tool0, origin xyz=0 0.1 0 rpy=-1.57079632679 0 0
- added joint limb_2_base_joint: type fixed, parent base_link, child limb_2_base_link, origin xyz=0.0 -0.1 0.0 rpy=0 1.5707963267948966 4.71238898038469
- added joint limb_2_ee_fixed_joint: type fixed, parent limb_2_wrist_3_link, child limb_2_ee_link, origin xyz=0.0 0.1 0.0 rpy=0.0 0.0 1.57079632679
- added joint limb_2_elbow_joint: type revolute, parent limb_2_upper_arm_link, child limb_2_forearm_link, origin xyz=0.0 -0.131 0.425 rpy=0.0 0.0 0.0, axis 0 1 0, limit lower=-3.14159265359 upper=3.14159265359 effort=150.0 velocity=3.14
- added joint limb_2_shoulder_lift_joint: type revolute, parent limb_2_shoulder_link, child limb_2_upper_arm_link, origin xyz=0.0 0.138 0.0 rpy=0.0 1.57079632679 0.0, axis 0 1 0, limit lower=-6.28318530718 upper=6.28318530718 effort=150.0 velocity=3.14
- added joint limb_2_shoulder_pan_joint: type revolute, parent limb_2_base_link, child limb_2_shoulder_link, origin xyz=0.0 0.0 0.163 rpy=0.0 0.0 0.0, axis 0 0 1, limit lower=-6.28318530718 upper=6.28318530718 effort=150.0 velocity=3.14
- added joint limb_2_wrist_1_joint: type revolute, parent limb_2_forearm_link, child limb_2_wrist_1_link, origin xyz=0.0 0.0 0.392 rpy=0.0 1.57079632679 0.0, axis 0 1 0, limit lower=-6.28318530718 upper=6.28318530718 effort=28.0 velocity=6.28
- added joint limb_2_wrist_2_joint: type revolute, parent limb_2_wrist_1_link, child limb_2_wrist_2_link, origin xyz=0.0 0.127 0.0 rpy=0.0 0.0 0.0, axis 0 0 1, limit lower=-6.28318530718 upper=6.28318530718 effort=28.0 velocity=6.28
- added joint limb_2_wrist_3_joint: type revolute, parent limb_2_wrist_2_link, child limb_2_wrist_3_link, origin xyz=0.0 0.0 0.1 rpy=0.0 0.0 0.0, axis 0 1 0, limit lower=-6.28318530718 upper=6.28318530718 effort=28.0 velocity=6.28
- added joint limb_2_wrist_3_link-tool0_fixed_joint: type fixed, parent limb_2_wrist_3_link, child limb_2_tool0, origin xyz=0 0.1 0 rpy=-1.57079632679 0 0

Commit message: Change base mass

File: mlivr_description/urdf/mlivr.urdf (robot description, URDF)
Before this commit: robot MLIVR, 19 links, 18 joints
Links:
- link base_link: mass 30.0 -> 20.0

File: mlivr_description/urdf/ur5e/mlivr.xacro (robot description, xacro)
@@ -7,7 +7,7 @@
   <link name="base_link">
     <inertial>
-      <mass value="30.0"/>
+      <mass value="20.0"/>
       <origin xyz="0 0 0" rpy="0 0 0"/>
-      <inertia ixx="0.2" ixy="0.0" ixz="0.0" iyy="0.2" iyz="0.0" izz="0.2"/>
+      <inertia ixx="0.133333" ixy="0.0" ixz="0.0" iyy="0.133333" iyz="0.0" izz="0.133333"/>
     </inertial>
     <visual>

Commit message: Visualize real and planned robot model and planned ee traj in rviz

File: mlivr_description/urdf/mlivr.urdf (robot description, URDF)
Before this commit: robot MLIVR, 19 links, 18 joints
Links:
- link limb_1_base_link: geometry collision mesh filename=package://mlivr_description/meshes/ur5e/collision/base.stl scale=1.0 1.0 1.0; visual mesh filename=package://mlivr_description/meshes/ur5e/visual/base.dae
- link limb_1_forearm_link: geometry collision mesh filename=package://mlivr_description/meshes/ur5e/collision/forearm.s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 scale=1.0 1.0 1.0; visual mesh filename=package://mlivr_description/meshes/ur5e/visual/forearm.dae
- link limb_1_shoulder_link: geometry collision mesh filename=package://mlivr_description/meshes/ur5e/collision/shoulder.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 scale=1.0 1.0 1.0; visual mesh filename=package://mlivr_description/meshes/ur5e/visual/shoulder.dae
- link limb_1_upper_arm_link: geometry collision mesh filename=package://mlivr_description/meshes/ur5e/collision/upperarm.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 scale=1.0 1.0 1.0; visual mesh filename=package://mlivr_description/meshes/ur5e/visual/upperarm.dae
- link limb_1_wrist_1_link: geometry collision mesh filename=package://mlivr_description/meshes/ur5e/collision/wrist1.stl scale=1.0 1.0 1.0; visual mesh filename=package://mlivr_description/meshes/ur5e/visual/wrist1.dae
- link limb_1_wrist_2_link: geometry collision mesh filename=package://mlivr_description/meshes/ur5e/collision/wrist2.stl scale=1.0 1.0 1.0; visual mesh filename=package://mlivr_description/meshes/ur5e/visual/wrist2.dae
- link limb_1_wrist_3_link: geometry collision mesh filename=package://mlivr_description/meshes/ur5e/collision/wrist3.stl scale=1.0 1.0 1.0; visual mesh filename=package://mlivr_description/meshes/ur5e/visual/wrist3.dae
- link limb_2_base_link: geometry collision mesh filename=package://mlivr_description/meshes/ur5e/collision/base.stl scale=1.0 1.0 1.0; visual mesh filename=package://mlivr_description/meshes/ur5e/visual/base.dae
- link limb_2_forearm_link: geometry collision mesh filename=package://mlivr_description/meshes/ur5e/collision/forearm.s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 scale=1.0 1.0 1.0; visual mesh filename=package://mlivr_description/meshes/ur5e/visual/forearm.dae
- link limb_2_shoulder_link: geometry collision mesh filename=package://mlivr_description/meshes/ur5e/collision/shoulder.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 scale=1.0 1.0 1.0; visual mesh filename=package://mlivr_description/meshes/ur5e/visual/shoulder.dae
- link limb_2_upper_arm_link: geometry collision mesh filename=package://mlivr_description/meshes/ur5e/collision/upperarm.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 scale=1.0 1.0 1.0; visual mesh filename=package://mlivr_description/meshes/ur5e/visual/upperarm.dae
- link limb_2_wrist_1_link: geometry collision mesh filename=package://mlivr_description/meshes/ur5e/collision/wrist1.stl scale=1.0 1.0 1.0; visual mesh filename=package://mlivr_description/meshes/ur5e/visual/wrist1.dae
- link limb_2_wrist_2_link: geometry collision mesh filename=package://mlivr_description/meshes/ur5e/collision/wrist2.stl scale=1.0 1.0 1.0; visual mesh filename=package://mlivr_description/meshes/ur5e/visual/wrist2.dae
- link limb_2_wrist_3_link: geometry collision mesh filename=package://mlivr_description/meshes/ur5e/collision/wrist3.stl scale=1.0 1.0 1.0; visual mesh filename=package://mlivr_description/meshes/ur5e/visual/wrist3.dae

File: mlivr_description/urdf/ur5e/mlivr.xacro (robot description, xacro)
@@ -1,4 +1,5 @@
 <?xml version="1.0"?>
 <robot name="MLIVR" xmlns:xacro="http://www.ros.org/wiki/xacro">
+  <xacro:arg name="mesh_dir" default="package://mlivr_description/meshes"/>
   <xacro:include filename="./ur5e_macro.xacro"/>
   <mujoco>

Commit message: Change robot model

File: mlivr_description/urdf/mlivr.urdf (robot description, URDF)
Before this commit: robot MLIVR, 19 links, 18 joints
Links:
- removed link limb_1_ee_link
- removed link limb_1_tool0
- removed link limb_2_ee_link
- removed link limb_2_tool0
- added link limb_1_gripper_link, mass 0.5; collision cylinder length=0.05 radius=0.03; visual cylinder length=0.05 radius=0.03
- added link limb_1_palm_link
- added link limb_2_gripper_link, mass 0.5; collision cylinder length=0.05 radius=0.03; visual cylinder length=0.05 radius=0.03
- added link limb_2_palm_link
Joints:
- removed joint limb_1_wrist_3_link-tool0_fixed_joint
- removed joint limb_2_wrist_3_link-tool0_fixed_joint
- added joint limb_1_palm_fixed_joint: type fixed, parent limb_1_gripper_link, child limb_1_palm_link, origin xyz=0 0 0.05 rpy=0 0 0
- added joint limb_2_palm_fixed_joint: type fixed, parent limb_2_gripper_link, child limb_2_palm_link, origin xyz=0 0 0.05 rpy=0 0 0
- joint limb_1_ee_fixed_joint: child limb_1_ee_link -> limb_1_gripper_link; origin xyz=0.0 0.1 0.0 rpy=0.0 0.0 1.57079632679 -> xyz=0 0.099 0 rpy=-1.5707963267948966 0 0
- joint limb_2_ee_fixed_joint: child limb_2_ee_link -> limb_2_gripper_link; origin xyz=0.0 0.1 0.0 rpy=0.0 0.0 1.57079632679 -> xyz=0 0.099 0 rpy=-1.5707963267948966 0 0

File: mlivr_description/urdf/ur5e/mlivr.xacro (robot description, xacro)
@@ -3,4 +3,5 @@
   <xacro:arg name="mesh_dir" default="package://mlivr_description/meshes"/>
   <xacro:include filename="./ur5e_macro.xacro"/>
+  <xacro:include filename="./mlivr_gripper.xacro"/>
   <mujoco>
     <compiler strippath="false"/>
@@ -29,6 +30,8 @@
     <origin xyz="0.0 0.1 0.0" rpy="0 ${radians(90)} ${radians(90)}"/>
   </xacro:ur5e>
+  <xacro:mlivr_gripper prefix="limb_1"/>
   <xacro:ur5e prefix="limb_2" parent="base_link">
     <origin xyz="0.0 -0.1 0.0" rpy="0 ${radians(90)} ${radians(270)}"/>
   </xacro:ur5e>
+  <xacro:mlivr_gripper prefix="limb_2"/>
 </robot>

File: mlivr_description/urdf/ur5e/ur5e_macro.xacro (robot description, xacro)
@@ -196,23 +196,4 @@
       </collision>
     </link>
-    <joint name="${prefix}_ee_fixed_joint" type="fixed">
-      <parent link="${prefix}_wrist_3_link"/>
-      <child link="${prefix}_ee_link"/>
-      <origin rpy="0.0 0.0 1.57079632679" xyz="0.0 0.1 0.0"/>
-    </joint>
-    <link name="${prefix}_ee_link">
-      <collision>
-        <geometry>
-          <box size="0.01 0.01 0.01"/>
-        </geometry>
-        <origin rpy="0 0 0" xyz="-0.01 0 0"/>
-      </collision>
-    </link>
-    <link name="${prefix}_tool0"/>
-    <joint name="${prefix}_wrist_3_link-tool0_fixed_joint" type="fixed">
-      <origin rpy="-1.57079632679 0 0" xyz="0 0.1 0"/>
-      <parent link="${prefix}_wrist_3_link"/>
-      <child link="${prefix}_tool0"/>
-    </joint>
   </xacro:macro>
 </robot>
