Commit message: Feature/reaction aware traj opt (#1)
* Change to multi-phase

* Implement impulse model

* Add impact minimization const

* Add state constraint

* minor change

* Remove active_contacts and impulse model

* Merge branch 'feature/changeRobotModel'

* Change ee displacement

* Change init state

* Change base mass

* Change state reg cost

* Add via point and floor collision cost

* Remove supporting frame from collision list

* Add mid point of spline for gj control

* Add FT sensor and publish data

* Change grasp interface from seattrack to handrail

* Change init state (and cost weight)

* minor change

* Change frame of displacement to world frame

* Change horizon step num

* Visualize frame, contact force and contact point

* minor change

* Add ee vel cost

* Add external collision weight in yaml

* tune cost weight

* Change damping and fricitionloss in xml

* Change pd gain

* Change pd gain

* Add pd gain setting in yaml

* Refactor sim node

* Change to mjcb_control

* Change to torque control for TO

* Change var type for gj control

* Visualize real and planned robot model and planned ee traj in rviz

* Publish odom topic

* Subscribe odom topic

* Update collision cost computation

* minor change

* Update README

* Add trigger and traj visualization for gj sim

* bugfix for gj

* Merge branch 'feature/designCost'

* Create base_controller

* Modified wb_control

* Update publishTargetTF

* Create kinematic jacobian control

* Change file extension

* Change dir

* Plot graphs for kj

* Change robot model

* Update init state

* Modify model

* Rename ft sensor frame id

* minor change

* Change joint params in mjcf

* Change weights

* Update model param

* Record rosbag and plot graphs

* Implement momentum distribution

* Create computeInertiaMatrices

* Update momentum_distribution

* Create ramp_control

* minor change

* Create low_reaction_swing_trajectory and include NLopt

* Add solveNumericalIK

* Update lrst

* Remove mlivr_model dependency

* Remove dependency

* Generate optimized trajectory by LRST

* Plot

* Create member var

* Update comments

* Separate struct

* Create yaml for ramp

* Use ros2 params

* Update generateTrajectory

* Update ros2 params

* Tune weights

* Add params for momentum distribution factor

* Publish planned TF

* Get data

* Remove old data

* Get data

* Add armature and damping params

* Change control reg cost and weights

* Change weights

* Get data

* Update swing joint names

* Remove mlivr_model

* Get data

* minor change

* Create WeightScheduleParams and computeWeightMultiplier

* refactor

* Use free fwddyn

* Remove ramp pkg

* Update ramp_control

* Get trigger time

* Update wb_control

* Move dir

* Update ramp_control

* Update ramp_control

* Change robot base and gripper color

* Success: stride 1m

Add iss_jem.dae files

Add iss_jem.dae files

Create env_visualizer

minor change

Change brightness

Add dae of light ver

Add seattrack 2

Add init_grasp 2

Remove large size dae files

* Update gitignore

* Update init state

* Success: stride 0.5

* Try gj case

* Try ramp case

* Update kj and gj

* Update init gait

* Redesign cost and tune weight

* minor change

* Remove arch for cost

* minor change

* Refactor cost functions

* Add ActivationModelWeightedQuad for state and ee tracking

* Add elbow joint limit cost (for self collision avoidance)

* minor change

* Add base_pose_reg_diag

* Tune weight

* Change elbow joint limit

* Change init base height

* minor change

* Case 2 data

* Add case: ee move to wall

* Case 1 params

* Remove old data

* Get data of case 1

* Rename launch files

* Case 3 params

* Get case 3 data

* Update model

* Get case 1 data for RAMP-PMD

* Add base ang dist data

* Add baseline data for case 1

* Get case 1 data

* Move dir

* Remove case 1 data (linear traj)

* Get case 1 data with 0.1m step height

* Get case 2 data of baseline

* Rename file

* fix duration for plot

* Change plot

File: mlivr_description/urdf/mlivr.urdf (robot description, URDF)
Before this commit: robot MLIVR, 21 links, 20 joints
Links:
- removed link limb_1_link_0
- removed link limb_1_link_1
- removed link limb_1_link_2
- removed link limb_1_link_3
- removed link limb_1_link_4
- removed link limb_1_link_5
- removed link limb_1_link_6
- removed link limb_1_link_7
- removed link limb_1_link_ee
- removed link limb_1_link_gripper
- removed link limb_2_link_0
- removed link limb_2_link_1
- removed link limb_2_link_2
- removed link limb_2_link_3
- removed link limb_2_link_4
- removed link limb_2_link_5
- removed link limb_2_link_6
- removed link limb_2_link_7
- removed link limb_2_link_ee
- removed link limb_2_link_gripper
- added link limb_1_base_link, mass 4.0; collision mesh filename=package://mlivr_description/meshes/ur5e/collision/base.stl scale=1.0 1.0 1.0; visual mesh filename=package://mlivr_description/meshes/ur5e/visual/base.dae
- added link limb_1_forearm_link, mass 2.275; collision mesh filename=package://mlivr_description/meshes/ur5e/collision/forearm.s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 scale=1.0 1.0 1.0; visual mesh filename=package://mlivr_description/meshes/ur5e/visual/forearm.dae
- added link limb_1_gripper_link, mass 0.5; collision cylinder length=0.05 radius=0.03; visual cylinder length=0.05 radius=0.03
- added link limb_1_palm_link
- added link limb_1_shoulder_link, mass 3.7; collision mesh filename=package://mlivr_description/meshes/ur5e/collision/shoulder.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 scale=1.0 1.0 1.0; visual mesh filename=package://mlivr_description/meshes/ur5e/visual/shoulder.dae
- added link limb_1_upper_arm_link, mass 8.393; collision mesh filename=package://mlivr_description/meshes/ur5e/collision/upperarm.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 scale=1.0 1.0 1.0; visual mesh filename=package://mlivr_description/meshes/ur5e/visual/upperarm.dae
- added link limb_1_wrist_1_link, mass 1.219; collision mesh filename=package://mlivr_description/meshes/ur5e/collision/wrist1.stl scale=1.0 1.0 1.0; visual mesh filename=package://mlivr_description/meshes/ur5e/visual/wrist1.dae
- added link limb_1_wrist_2_link, mass 1.219; collision mesh filename=package://mlivr_description/meshes/ur5e/collision/wrist2.stl scale=1.0 1.0 1.0; visual mesh filename=package://mlivr_description/meshes/ur5e/visual/wrist2.dae
- added link limb_1_wrist_3_link, mass 0.1879; collision mesh filename=package://mlivr_description/meshes/ur5e/collision/wrist3.stl scale=1.0 1.0 1.0; visual mesh filename=package://mlivr_description/meshes/ur5e/visual/wrist3.dae
- added link limb_2_base_link, mass 4.0; collision mesh filename=package://mlivr_description/meshes/ur5e/collision/base.stl scale=1.0 1.0 1.0; visual mesh filename=package://mlivr_description/meshes/ur5e/visual/base.dae
- added link limb_2_forearm_link, mass 2.275; collision mesh filename=package://mlivr_description/meshes/ur5e/collision/forearm.s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 scale=1.0 1.0 1.0; visual mesh filename=package://mlivr_description/meshes/ur5e/visual/forearm.dae
- added link limb_2_gripper_link, mass 0.5; collision cylinder length=0.05 radius=0.03; visual cylinder length=0.05 radius=0.03
- added link limb_2_palm_link
- added link limb_2_shoulder_link, mass 3.7; collision mesh filename=package://mlivr_description/meshes/ur5e/collision/shoulder.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 scale=1.0 1.0 1.0; visual mesh filename=package://mlivr_description/meshes/ur5e/visual/shoulder.dae
- added link limb_2_upper_arm_link, mass 8.393; collision mesh filename=package://mlivr_description/meshes/ur5e/collision/upperarm.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 scale=1.0 1.0 1.0; visual mesh filename=package://mlivr_description/meshes/ur5e/visual/upperarm.dae
- added link limb_2_wrist_1_link, mass 1.219; collision mesh filename=package://mlivr_description/meshes/ur5e/collision/wrist1.stl scale=1.0 1.0 1.0; visual mesh filename=package://mlivr_description/meshes/ur5e/visual/wrist1.dae
- added link limb_2_wrist_2_link, mass 1.219; collision mesh filename=package://mlivr_description/meshes/ur5e/collision/wrist2.stl scale=1.0 1.0 1.0; visual mesh filename=package://mlivr_description/meshes/ur5e/visual/wrist2.dae
- added link limb_2_wrist_3_link, mass 0.1879; collision mesh filename=package://mlivr_description/meshes/ur5e/collision/wrist3.stl scale=1.0 1.0 1.0; visual mesh filename=package://mlivr_description/meshes/ur5e/visual/wrist3.dae
- link base_link: mass 50.0 -> 20.0; geometry collision box size=0.2 0.2 0.2; visual box size=0.2 0.2 0.2
Joints:
- removed joint base_link_limb_1_joint
- removed joint base_link_limb_2_joint
- removed joint limb_1_joint_1
- removed joint limb_1_joint_2
- removed joint limb_1_joint_3
- removed joint limb_1_joint_4
- removed joint limb_1_joint_5
- removed joint limb_1_joint_6
- removed joint limb_1_joint_7
- removed joint limb_1_joint_ee
- removed joint limb_1_joint_gripper
- removed joint limb_2_joint_1
- removed joint limb_2_joint_2
- removed joint limb_2_joint_3
- removed joint limb_2_joint_4
- removed joint limb_2_joint_5
- removed joint limb_2_joint_6
- removed joint limb_2_joint_7
- removed joint limb_2_joint_ee
- removed joint limb_2_joint_gripper
- added joint limb_1_base_joint: type fixed, parent base_link, child limb_1_base_link, origin xyz=0.0 0.1 0.0 rpy=0 1.5707963267948966 1.5707963267948966
- added joint limb_1_ee_fixed_joint: type fixed, parent limb_1_wrist_3_link, child limb_1_gripper_link, origin xyz=0 0.099 0 rpy=-1.5707963267948966 0 0
- added joint limb_1_elbow_joint: type revolute, parent limb_1_upper_arm_link, child limb_1_forearm_link, origin xyz=0.0 -0.131 0.425 rpy=0.0 0.0 0.0, axis 0 1 0, limit lower=-3.14159265359 upper=3.14159265359 effort=150.0 velocity=3.14
- added joint limb_1_palm_fixed_joint: type fixed, parent limb_1_gripper_link, child limb_1_palm_link, origin xyz=0 0 0.05 rpy=0 0 0
- added joint limb_1_shoulder_lift_joint: type revolute, parent limb_1_shoulder_link, child limb_1_upper_arm_link, origin xyz=0.0 0.138 0.0 rpy=0.0 1.57079632679 0.0, axis 0 1 0, limit lower=-6.28318530718 upper=6.28318530718 effort=150.0 velocity=3.14
- added joint limb_1_shoulder_pan_joint: type revolute, parent limb_1_base_link, child limb_1_shoulder_link, origin xyz=0.0 0.0 0.163 rpy=0.0 0.0 0.0, axis 0 0 1, limit lower=-6.28318530718 upper=6.28318530718 effort=150.0 velocity=3.14
- added joint limb_1_wrist_1_joint: type revolute, parent limb_1_forearm_link, child limb_1_wrist_1_link, origin xyz=0.0 0.0 0.392 rpy=0.0 1.57079632679 0.0, axis 0 1 0, limit lower=-6.28318530718 upper=6.28318530718 effort=28.0 velocity=6.28
- added joint limb_1_wrist_2_joint: type revolute, parent limb_1_wrist_1_link, child limb_1_wrist_2_link, origin xyz=0.0 0.127 0.0 rpy=0.0 0.0 0.0, axis 0 0 1, limit lower=-6.28318530718 upper=6.28318530718 effort=28.0 velocity=6.28
- added joint limb_1_wrist_3_joint: type revolute, parent limb_1_wrist_2_link, child limb_1_wrist_3_link, origin xyz=0.0 0.0 0.1 rpy=0.0 0.0 0.0, axis 0 1 0, limit lower=-6.28318530718 upper=6.28318530718 effort=28.0 velocity=6.28
- added joint limb_2_base_joint: type fixed, parent base_link, child limb_2_base_link, origin xyz=0.0 -0.1 0.0 rpy=0 1.5707963267948966 4.71238898038469
- added joint limb_2_ee_fixed_joint: type fixed, parent limb_2_wrist_3_link, child limb_2_gripper_link, origin xyz=0 0.099 0 rpy=-1.5707963267948966 0 0
- added joint limb_2_elbow_joint: type revolute, parent limb_2_upper_arm_link, child limb_2_forearm_link, origin xyz=0.0 -0.131 0.425 rpy=0.0 0.0 0.0, axis 0 1 0, limit lower=-3.14159265359 upper=3.14159265359 effort=150.0 velocity=3.14
- added joint limb_2_palm_fixed_joint: type fixed, parent limb_2_gripper_link, child limb_2_palm_link, origin xyz=0 0 0.05 rpy=0 0 0
- added joint limb_2_shoulder_lift_joint: type revolute, parent limb_2_shoulder_link, child limb_2_upper_arm_link, origin xyz=0.0 0.138 0.0 rpy=0.0 1.57079632679 0.0, axis 0 1 0, limit lower=-6.28318530718 upper=6.28318530718 effort=150.0 velocity=3.14
- added joint limb_2_shoulder_pan_joint: type revolute, parent limb_2_base_link, child limb_2_shoulder_link, origin xyz=0.0 0.0 0.163 rpy=0.0 0.0 0.0, axis 0 0 1, limit lower=-6.28318530718 upper=6.28318530718 effort=150.0 velocity=3.14
- added joint limb_2_wrist_1_joint: type revolute, parent limb_2_forearm_link, child limb_2_wrist_1_link, origin xyz=0.0 0.0 0.392 rpy=0.0 1.57079632679 0.0, axis 0 1 0, limit lower=-6.28318530718 upper=6.28318530718 effort=28.0 velocity=6.28
- added joint limb_2_wrist_2_joint: type revolute, parent limb_2_wrist_1_link, child limb_2_wrist_2_link, origin xyz=0.0 0.127 0.0 rpy=0.0 0.0 0.0, axis 0 0 1, limit lower=-6.28318530718 upper=6.28318530718 effort=28.0 velocity=6.28
- added joint limb_2_wrist_3_joint: type revolute, parent limb_2_wrist_2_link, child limb_2_wrist_3_link, origin xyz=0.0 0.0 0.1 rpy=0.0 0.0 0.0, axis 0 1 0, limit lower=-6.28318530718 upper=6.28318530718 effort=28.0 velocity=6.28
